File: ADuM_I2C_v3_arr2x4.kicad_pcb (KiCad board)
At the start: 4 copper layers, 50 x 50 mm, 0 parts

Commit message: Переделана панелизация платы ADuM_I2C_v3
Other:
- board outline removed

Commit message: Сформирован перечень элементов, 3D-модель, исправлены ошибки, реализована панелизация платы.
Routing:
- net /SCLq: track 16.2 -> 0.00 mm
- net /SCL: track 11.5 -> 0.00 mm
- net Net-(Q4-Pad2): track 11.1 -> 0.00 mm
- net /SDAq: track 10.1 -> 0.00 mm
- net Net-(Q7-Pad2): track 9.68 -> 0.00 mm
- net /SDA: track 9.09 -> 0.00 mm
- net Net-(Q8-Pad2): track 7.65 -> 0.00 mm
- net Net-(Q2-Pad2): track 7.62 -> 0.00 mm
- net Net-(Q6-Pad2): track 7.23 -> 0.00 mm
- net Net-(Q3-Pad2): track 6.48 -> 0.00 mm
- net Net-(Q1-Pad2): track 2.55 -> 0.00 mm
- net Net-(Q5-Pad2): track 1.84 -> 0.00 mm
Changed lines of the file:
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@@
     (thickness 1.6)
     (drawings 48)
-    (tracks 62)
+    (tracks 0)
     (zones 0)
     (modules 0)
-    (nets 13)
+    (nets 1)
   )
   (page A4)
@@
   )
   (net 0 "")
-  (net 1 /SCL)
-  (net 2 /SDA)
-  (net 3 /SCLq)
-  (net 4 /SDAq)
-  (net 5 "Net-(Q1-Pad2)")
-  (net 6 "Net-(Q2-Pad2)")
-  (net 7 "Net-(Q3-Pad2)")
-  (net 8 "Net-(Q4-Pad2)")
-  (net 9 "Net-(Q5-Pad2)")
-  (net 10 "Net-(Q6-Pad2)")
-  (net 11 "Net-(Q7-Pad2)")
-  (net 12 "Net-(Q8-Pad2)")
   (net_class Default "Это класс цепей по умолчанию."
     (clearance 0.2)
@@
     (uvia_dia 0.3)
     (uvia_drill 0.1)
-    (add_net /SCL)
-    (add_net /SCLq)
-    (add_net /SDA)
-    (add_net /SDAq)
-    (add_net "Net-(Q1-Pad2)")
-    (add_net "Net-(Q2-Pad2)")
-    (add_net "Net-(Q3-Pad2)")
-    (add_net "Net-(Q4-Pad2)")
-    (add_net "Net-(Q5-Pad2)")
-    (add_net "Net-(Q6-Pad2)")
-    (add_net "Net-(Q7-Pad2)")
-    (add_net "Net-(Q8-Pad2)")
   )
   (net_class Digital ""
@@
   (gr_line (start 74.5 48.5) (end 74.5 61) (layer Dwgs.User) (width 0.1))
   (gr_line (start 49.5 61) (end 74.5 61) (layer Dwgs.User) (width 0.1))
-  (segment (start 71.055999 59.564001) (end 71.906 58.714) (width 0.3) (layer In1.Cu) (net 1))
-  (segment (start 70.227999 59.564001) (end 71.055999 59.564001) (width 0.3) (layer In1.Cu) (net 1))
-  (segment (start 69.785999 58.752999) (end 69.785999 59.122001) (width 0.3) (layer In1.Cu) (net 1))
-  (segment (start 66.826 55.793) (end 69.785999 58.752999) (width 0.3) (layer In1.Cu) (net 1))
-  (segment (start 69.785999 59.122001) (end 70.227999 59.564001) (width 0.3) (layer In1.Cu) (net 1))
-  (segment (start 65.750781 55.793) (end 66.826 55.793) (width 0.3) (layer In1.Cu) (net 1))
-  (segment (start 63.903419 53.945638) (end 65.750781 55.793) (width 0.3) (layer In1.Cu) (net 1))
-  (segment (start 63.903419 53.379953) (end 63.903419 53.945638) (width 0.3) (layer In1.Cu) (net 1))
-  (segment (start 64.90299 54.12399) (end 64.90299 53.409645) (width 0.3) (layer In1.Cu) (net 2))
-  (segment (start 66.07199 55.29299) (end 64.90299 54.12399) (width 0.3) (layer In1.Cu) (net 2))
-  (segment (start 67.08799 55.29299) (end 66.07199 55.29299) (width 0.3) (layer In1.Cu) (net 2))
-  (segment (start 68.35 56.555) (end 67.08799 55.29299) (width 0.3) (layer In1.Cu) (net 2))
-  (segment (start 71.017 56.555) (end 68.35 56.555) (width 0.3) (layer In1.Cu) (net 2))
-  (segment (start 71.906 57.444) (end 71.017 56.555) (width 0.3) (layer In1.Cu) (net 2))
-  (segment (start 52.944001 59.564001) (end 52.094 58.714) (width 0.3) (layer In1.Cu) (net 3))
-  (segment (start 53.772001 59.564001) (end 52.944001 59.564001) (width 0.3) (layer In1.Cu) (net 3))
-  (segment (start 52.105998 58.714) (end 52.955999 59.564001) (width 0.3) (layer In1.Cu) (net 3))
-  (segment (start 52.955999 59.564001) (end 53.772001 59.564001) (width 0.3) (layer In1.Cu) (net 3))
-  (segment (start 52.094 58.714) (end 52.105998 58.714) (width 0.3) (layer In1.Cu) (net 3))
-  (segment (start 60.11014 50.685578) (end 60.11014 50.590919) (width 0.3) (layer In1.Cu) (net 3))
-  (segment (start 59.470248 51.32547) (end 60.11014 50.685578) (width 0.3) (layer In1.Cu) (net 3))
-  (segment (start 54.253 55.698998) (end 58.626528 51.32547) (width 0.3) (layer In1.Cu) (net 3))
-  (segment (start 58.626528 51.32547) (end 59.470248 51.32547) (width 0.3) (layer In1.Cu) (net 3))
-  (segment (start 54.253 59.083002) (end 54.253 55.698998) (width 0.3) (layer In1.Cu) (net 3))
-  (segment (start 53.772001 59.564001) (end 54.253 59.083002) (width 0.3) (layer In1.Cu) (net 3))
-  (segment (start 58.544562 50.575469) (end 59.110247 50.575469) (width 0.3) (layer In1.Cu) (net 4))
-  (segment (start 52.094 57.026032) (end 58.544562 50.575469) (width 0.3) (layer In1.Cu) (net 4))
-  (segment (start 52.094 57.444) (end 52.094 57.026032) (width 0.3) (layer In1.Cu) (net 4))
-  (segment (start 67.302898 55.316102) (end 67.302898 54.523004) (width 0.3) (layer In2.Cu) (net 5))
-  (segment (start 66.064 56.555) (end 67.302898 55.316102) (width 0.3) (layer In2.Cu) (net 5))
-  (segment (start 66.064 58.587) (end 65.498315 58.587) (width 0.3) (layer In2.Cu) (net 6))
-  (segment (start 65.498315 58.587) (end 65.313999 58.402684) (width 0.3) (layer In2.Cu) (net 6))
-  (segment (start 65.313999 58.402684) (end 65.313999 56.194999) (width 0.3) (layer In2.Cu) (net 6))
-  (segment (start 65.313999 56.194999) (end 65.653631 55.855367) (width 0.3) (layer In2.Cu) (net 6))
-  (segment (start 65.653631 55.855367) (end 65.653631 52.331594) (width 0.3) (layer In2.Cu) (net 6))
-  (segment (start 65.653631 52.331594) (end 65.241533 51.919496) (width 0.3) (layer In2.Cu) (net 6))
-  (segment (start 70.000994 55.607008) (end 70.000994 54.269) (width 0.3) (layer In2.Cu) (net 7))
-  (segment (start 67.567001 58.041001) (end 70.000994 55.607008) (width 0.3) (layer In2.Cu) (net 7))
-  (segment (start 66.846999 58.041001) (end 67.567001 58.041001) (width 0.3) (layer In2.Cu) (net 7))
-  (segment (start 66.376998 57.571) (end 66.846999 58.041001) (width 0.3) (layer In2.Cu) (net 7))
-  (segment (start 66.064 57.571) (end 66.376998 57.571) (width 0.3) (layer In2.Cu) (net 7))
-  (segment (start 70.763 53.373807) (end 72.214811 51.921996) (width 0.3) (layer In2.Cu) (net 8))
-  (segment (start 70.763 55.552122) (end 70.763 53.373807) (width 0.3) (layer In2.Cu) (net 8))
-  (segment (start 67.957001 58.358121) (end 70.763 55.552122) (width 0.3) (layer In2.Cu) (net 8))
-  (segment (start 67.957001 59.201001) (end 67.957001 58.358121) (width 0.3) (layer In2.Cu) (net 8))
-  (segment (start 67.555002 59.603) (end 67.957001 59.201001) (width 0.3) (layer In2.Cu) (net 8))
-  (segment (start 66.064 59.603) (end 67.555002 59.603) (width 0.3) (layer In2.Cu) (net 8))
-  (segment (start 57.955124 56.561379) (end 57.957705 56.561379) (width 0.3) (layer In2.Cu) (net 9))
-  (segment (start 56.65401 55.260265) (end 57.955124 56.561379) (width 0.3) (layer In2.Cu) (net 9))
-  (segment (start 58.501685 58.587) (end 57.936 58.587) (width 0.3) (layer In2.Cu) (net 10))
-  (segment (start 58.952 58.136685) (end 58.501685 58.587) (width 0.3) (layer In2.Cu) (net 10))
-  (segment (start 58.952 52.11) (end 58.952 58.136685) (width 0.3) (layer In2.Cu) (net 10))
-  (segment (start 57.841998 57.571) (end 57.936 57.571) (width 0.3) (layer In2.Cu) (net 11))
-  (segment (start 57.371997 58.041001) (end 57.841998 57.571) (width 0.3) (layer In2.Cu) (net 11))
-  (segment (start 56.432999 58.041001) (end 57.371997 58.041001) (width 0.3) (layer In2.Cu) (net 11))
-  (segment (start 51.784577 53.392579) (end 56.432999 58.041001) (width 0.3) (layer In2.Cu) (net 11))
-  (segment (start 51.784577 51.982726) (end 51.784577 53.392579) (width 0.3) (layer In2.Cu) (net 11))
-  (segment (start 56.042999 58.492997) (end 56.042999 59.201001) (width 0.3) (layer In2.Cu) (net 12))
-  (segment (start 56.474133 59.632135) (end 57.935957 59.632135) (width 0.3) (layer In2.Cu) (net 12))
-  (segment (start 53.216002 55.666) (end 56.042999 58.492997) (width 0.3) (layer In2.Cu) (net 12))
-  (segment (start 56.042999 59.201001) (end 56.474133 59.632135) (width 0.3) (layer In2.Cu) (net 12))
-  (segment (start 52.348 55.666) (end 53.216002 55.666) (width 0.3) (layer In2.Cu) (net 12))
 )

Commit message: Созданы две панели: односторонняя и двухсторонняя, объединяющие все платы, кроме цифрового модуля. Добавлен окантовка по контуру платы с двух сторон и текст: "JLCJLCJLCJLC"
Routing:
- net /SCLq: track 0.00 -> 16.2 mm
- net /SCL: track 0.00 -> 11.5 mm
- net Net-(Q4-Pad2): track 0.00 -> 11.1 mm
- net /SDAq: track 0.00 -> 10.1 mm
- net Net-(Q7-Pad2): track 0.00 -> 9.68 mm
- net /SDA: track 0.00 -> 9.09 mm
- net Net-(Q8-Pad2): track 0.00 -> 7.65 mm
- net Net-(Q2-Pad2): track 0.00 -> 7.62 mm
- net Net-(Q6-Pad2): track 0.00 -> 7.23 mm
- net Net-(Q3-Pad2): track 0.00 -> 6.48 mm
- net Net-(Q1-Pad2): track 0.00 -> 2.55 mm
- net Net-(Q5-Pad2): track 0.00 -> 1.84 mm
Other:
- board outline added: 27 x 41.9 mm
