File: PCB_4x_pnlz1_3.kicad_pcb (KiCad board)
At the start: 4 copper layers, 50 x 76 mm, 300 parts, among them J1 A, J1 L_input, J1 Load2, J2 B, J2 Dig_mod_iface, J2 Pow_mng_pow, J3 Load1, J4 Load2, J5 SWD (PLS5), J6 Dig_mod_iface, K1 HFD2_005-S-L2-D_Split, K2 HFD2_005-S-L2-D_Split, Q1 2N5551S, Q1 BSS138, Q2 2N5551S, Q2 BSS138, Q3 BSS138, Q4 BSS138, Q5 2N5551S, Q5 BSS138, Q6 2N5551S, Q6 BSS138, Q7 BSS138, Q8 BSS138, U1 ADuM1251ARZ, U1 DC12003, U2 ADuM1201AR, U2 G3MB-202PL, U2 PCA9536DP, U3 G3MB-202PL, U4 DC5V_DC5V3V3_v3, U5 STM32F030F4Px, U6 HLW8112, U7 ADuM_I2C_v3, Y1 CSTCE8M, Y2 ABLS-3.579545MHZ-D-3-Y-T

Commit message: Последние изменения в BOM
Parts:
- removed the C1 at (95.2, 109.2)
- removed the C1 at (82.7, 109.2)
- removed the C1 at (70.2, 109.2)
- removed the C2 at (95.2, 110.7)
- removed the C2 at (82.7, 110.7)
- removed the C2 at (70.2, 110.7)
- removed the C3 at (95.2, 110.7)
- removed the C3 at (82.7, 110.7)
- removed the C3 at (70.2, 110.7)
- removed the C4 at (95.2, 121.1)
- removed the C4 at (82.7, 121.1)
- removed the C4 at (70.2, 121.1)
- removed the C5 at (95.2, 121.1)
- removed the C5 at (82.7, 121.1)
- removed the C5 at (70.2, 121.1)
- removed the C6 at (95.2, 122.6)
- removed the C6 at (82.7, 122.6)
- removed the C6 at (70.2, 122.6)
- removed the J1 at (94.5, 104.7)
- removed the J1 at (82.0, 104.7)
- removed the J1 at (69.5, 104.7)
- removed the J2 at (94.5, 124.5)
- removed the J2 at (82.0, 124.5)
- removed the J2 at (69.5, 124.5)
- removed the Q1 at (89.0, 113.0)
- removed the Q1 at (76.5, 113.0)
- removed the Q1 at (64.0, 113.0)
- removed the Q2 at (89.0, 113.0)
- removed the Q2 at (76.5, 113.0)
- removed the Q2 at (64.0, 113.0)
- removed the Q3 at (89.0, 105.4)
- removed the Q3 at (76.5, 105.4)
- removed the Q3 at (64.0, 105.4)
- removed the Q4 at (89.0, 105.4)
- removed the Q4 at (76.5, 105.4)
- removed the Q4 at (64.0, 105.4)
- removed the Q5 at (89.1, 118.8)
- removed the Q5 at (76.6, 118.8)
- removed the Q5 at (64.1, 118.8)
- removed the Q6 at (89.1, 118.8)
- removed the Q6 at (76.6, 118.8)
- removed the Q6 at (64.1, 118.8)
- removed the Q7 at (89.1, 126.4)
- removed the Q7 at (76.6, 126.4)
- removed the Q7 at (64.1, 126.4)
- removed the Q8 at (89.1, 126.4)
- removed the Q8 at (76.6, 126.4)
- removed the Q8 at (64.1, 126.4)
- removed the R1 at (86.4, 112.8)
- removed the R1 at (73.9, 112.8)
- removed the R1 at (61.4, 112.8)
- removed the R10 at (89.0, 110.4)
- removed the R10 at (76.5, 110.4)
- removed the R10 at (64.0, 110.4)
- removed the R11 at (89.0, 107.9)
- removed the R11 at (76.5, 107.9)
- removed the R11 at (64.0, 107.9)
- removed the R12 at (89.0, 107.9)
- removed the R12 at (76.5, 107.9)
- removed the R12 at (64.0, 107.9)
- removed the R13 at (89.0, 121.4)
- removed the R13 at (76.5, 121.4)
- removed the R13 at (64.0, 121.4)
- removed the R14 at (89.0, 121.4)
- removed the R14 at (76.5, 121.4)
- removed the R14 at (64.0, 121.4)
- removed the R15 at (89.0, 123.9)
- removed the R15 at (76.5, 123.9)
- removed the R15 at (64.0, 123.9)
- removed the R16 at (89.0, 123.9)
- removed the R16 at (76.5, 123.9)
- removed the R16 at (64.0, 123.9)
- removed the R17 at (91.6, 119.0)
- removed the R17 at (79.1, 119.0)
- removed the R17 at (66.6, 119.0)
- removed the R18 at (86.5, 119.0)
- removed the R18 at (74.0, 119.0)
- removed the R18 at (61.5, 119.0)
- removed the R19 at (86.5, 126.3)
- removed the R19 at (74.0, 126.3)
- removed the R19 at (61.5, 126.3)
- removed the R2 at (91.6, 112.8)
- removed the R2 at (79.1, 112.8)
- removed the R2 at (66.6, 112.8)
- removed the R20 at (91.6, 126.2)
- removed the R20 at (79.1, 126.2)
- removed the R20 at (66.6, 126.2)
- removed the R21 at (86.5, 119.0)
- removed the R21 at (74.0, 119.0)
- removed the R21 at (61.5, 119.0)
- removed the R22 at (91.6, 119.0)
- removed the R22 at (79.1, 119.0)
- removed the R22 at (66.6, 119.0)
- removed the R23 at (91.6, 126.2)
- removed the R23 at (79.1, 126.2)
- removed the R23 at (66.6, 126.2)
- removed the R24 at (86.5, 126.2)
- removed the R24 at (74.0, 126.2)
- removed the R24 at (61.5, 126.2)
- removed the R3 at (86.4, 105.5)
- removed the R3 at (73.9, 105.5)
- removed the R3 at (61.4, 105.5)
- removed the R4 at (91.6, 105.5)
- removed the R4 at (79.1, 105.5)
- removed the R4 at (66.6, 105.5)
- removed the R5 at (91.6, 112.8)
- removed the R5 at (79.1, 112.8)
- removed the R5 at (66.6, 112.8)
- removed the R6 at (86.4, 112.8)
- removed the R6 at (73.9, 112.8)
- removed the R6 at (61.4, 112.8)
- removed the R7 at (91.6, 105.5)
- removed the R7 at (79.1, 105.5)
- removed the R7 at (66.6, 105.5)
- removed the R8 at (86.4, 105.5)
- removed the R8 at (73.9, 105.5)
- removed the R8 at (61.4, 105.5)
- removed the R9 at (89.0, 110.4)
- removed the R9 at (76.5, 110.4)
- removed the R9 at (64.0, 110.4)
- removed the U1 at (95.2, 115.9)
- removed the U1 at (82.7, 115.9)
- removed the U1 at (70.2, 115.9)
- removed the U2 at (95.2, 115.9)
- removed the U2 at (82.7, 115.9)
- removed the U2 at (70.2, 115.9)
- added C1: 1uF, Capacitor_SMD:C_0603_1608Metric, B.Cu at (106.6, 110.2)
- added C1: 1uF, Capacitor_SMD:C_0603_1608Metric, B.Cu at (94.1, 110.2)
- added C1: 1uF, Capacitor_SMD:C_0603_1608Metric, B.Cu at (81.6, 110.2)
- added C2: 100nF, Capacitor_SMD:C_0603_1608Metric, B.Cu at (106.6, 111.7)
- added C2: 100nF, Capacitor_SMD:C_0603_1608Metric, B.Cu at (94.1, 111.7)
- added C2: 100nF, Capacitor_SMD:C_0603_1608Metric, B.Cu at (81.6, 111.7)
- added C3: 100nF, Capacitor_SMD:C_0603_1608Metric, F.Cu at (106.6, 111.7)
- added C3: 100nF, Capacitor_SMD:C_0603_1608Metric, F.Cu at (94.1, 111.7)
- added C3: 100nF, Capacitor_SMD:C_0603_1608Metric, F.Cu at (81.6, 111.7)
- added C4: 100nF, Capacitor_SMD:C_0603_1608Metric, B.Cu at (106.6, 122.1)
- added C4: 100nF, Capacitor_SMD:C_0603_1608Metric, B.Cu at (94.1, 122.1)
- added C4: 100nF, Capacitor_SMD:C_0603_1608Metric, B.Cu at (81.6, 122.1)
- added C5: 100nF, Capacitor_SMD:C_0603_1608Metric, F.Cu at (106.6, 122.1)
- added C5: 100nF, Capacitor_SMD:C_0603_1608Metric, F.Cu at (94.1, 122.1)
- added C5: 100nF, Capacitor_SMD:C_0603_1608Metric, F.Cu at (81.6, 122.1)
- added C6: 1uF, Capacitor_SMD:C_0603_1608Metric, B.Cu at (106.6, 123.6)
- added C6: 1uF, Capacitor_SMD:C_0603_1608Metric, B.Cu at (94.1, 123.6)
- added C6: 1uF, Capacitor_SMD:C_0603_1608Metric, B.Cu at (81.6, 123.6)
- added J1: A, Modules:PinHeader_2x03_P1.27mm_Horizontal_short, F.Cu at (105.9, 105.7)
- added J1: A, Modules:PinHeader_2x03_P1.27mm_Horizontal_short, F.Cu at (93.4, 105.7)
- added J1: A, Modules:PinHeader_2x03_P1.27mm_Horizontal_short, F.Cu at (80.9, 105.7)
- added J2: B, Modules:PinHeader_2x03_P1.27mm_Horizontal_short, F.Cu at (105.9, 125.5)
- added J2: B, Modules:PinHeader_2x03_P1.27mm_Horizontal_short, F.Cu at (93.4, 125.5)
- added J2: B, Modules:PinHeader_2x03_P1.27mm_Horizontal_short, F.Cu at (80.9, 125.5)
- added Q1: BSS138, Package_TO_SOT_SMD:SOT-23, B.Cu at (100.4, 114.0)
- added Q1: BSS138, Package_TO_SOT_SMD:SOT-23, B.Cu at (87.9, 114.0)
- added Q1: BSS138, Package_TO_SOT_SMD:SOT-23, B.Cu at (75.4, 114.0)
- added Q2: BSS138, Package_TO_SOT_SMD:SOT-23, F.Cu at (100.4, 114.0)
- added Q2: BSS138, Package_TO_SOT_SMD:SOT-23, F.Cu at (87.9, 114.0)
- added Q2: BSS138, Package_TO_SOT_SMD:SOT-23, F.Cu at (75.4, 114.0)
- added Q3: BSS138, Package_TO_SOT_SMD:SOT-23, F.Cu at (100.4, 106.4)
- added Q3: BSS138, Package_TO_SOT_SMD:SOT-23, F.Cu at (87.9, 106.4)
- added Q3: BSS138, Package_TO_SOT_SMD:SOT-23, F.Cu at (75.4, 106.4)
- added Q4: BSS138, Package_TO_SOT_SMD:SOT-23, B.Cu at (100.4, 106.4)
- added Q4: BSS138, Package_TO_SOT_SMD:SOT-23, B.Cu at (87.9, 106.4)
- added Q4: BSS138, Package_TO_SOT_SMD:SOT-23, B.Cu at (75.4, 106.4)
- added Q5: BSS138, Package_TO_SOT_SMD:SOT-23, F.Cu at (100.5, 119.8)
- added Q5: BSS138, Package_TO_SOT_SMD:SOT-23, F.Cu at (88.0, 119.8)
- added Q5: BSS138, Package_TO_SOT_SMD:SOT-23, F.Cu at (75.5, 119.8)
- added Q6: BSS138, Package_TO_SOT_SMD:SOT-23, B.Cu at (100.5, 119.8)
- added Q6: BSS138, Package_TO_SOT_SMD:SOT-23, B.Cu at (88.0, 119.8)
- added Q6: BSS138, Package_TO_SOT_SMD:SOT-23, B.Cu at (75.5, 119.8)
- added Q7: BSS138, Package_TO_SOT_SMD:SOT-23, F.Cu at (100.5, 127.4)
- added Q7: BSS138, Package_TO_SOT_SMD:SOT-23, F.Cu at (88.0, 127.4)
- added Q7: BSS138, Package_TO_SOT_SMD:SOT-23, F.Cu at (75.5, 127.4)
- added Q8: BSS138, Package_TO_SOT_SMD:SOT-23, B.Cu at (100.5, 127.4)
- added Q8: BSS138, Package_TO_SOT_SMD:SOT-23, B.Cu at (88.0, 127.4)
- added Q8: BSS138, Package_TO_SOT_SMD:SOT-23, B.Cu at (75.5, 127.4)
- added R1: 2.2M, Resistor_SMD:R_0603_1608Metric, B.Cu at (97.8, 113.8)
- added R1: 2.2M, Resistor_SMD:R_0603_1608Metric, B.Cu at (85.3, 113.8)
- added R1: 2.2M, Resistor_SMD:R_0603_1608Metric, B.Cu at (72.8, 113.8)
- added R10: 10k, Resistor_SMD:R_0603_1608Metric, F.Cu at (100.4, 111.4)
- added R10: 10k, Resistor_SMD:R_0603_1608Metric, F.Cu at (87.9, 111.4)
- added R10: 10k, Resistor_SMD:R_0603_1608Metric, F.Cu at (75.4, 111.4)
- added R11: 10k, Resistor_SMD:R_0603_1608Metric, F.Cu at (100.4, 108.9)
- added R11: 10k, Resistor_SMD:R_0603_1608Metric, F.Cu at (87.9, 108.9)
- added R11: 10k, Resistor_SMD:R_0603_1608Metric, F.Cu at (75.4, 108.9)
- added R12: 10k, Resistor_SMD:R_0603_1608Metric, B.Cu at (100.4, 108.9)
- added R12: 10k, Resistor_SMD:R_0603_1608Metric, B.Cu at (87.9, 108.9)
- added R12: 10k, Resistor_SMD:R_0603_1608Metric, B.Cu at (75.4, 108.9)
- added R13: 10k, Resistor_SMD:R_0603_1608Metric, F.Cu at (100.4, 122.4)
- added R13: 10k, Resistor_SMD:R_0603_1608Metric, F.Cu at (87.9, 122.4)
- added R13: 10k, Resistor_SMD:R_0603_1608Metric, F.Cu at (75.4, 122.4)
- added R14: 10k, Resistor_SMD:R_0603_1608Metric, B.Cu at (100.4, 122.4)
- added R14: 10k, Resistor_SMD:R_0603_1608Metric, B.Cu at (87.9, 122.4)
- added R14: 10k, Resistor_SMD:R_0603_1608Metric, B.Cu at (75.4, 122.4)
- added R15: 10k, Resistor_SMD:R_0603_1608Metric, F.Cu at (100.4, 124.9)
- added R15: 10k, Resistor_SMD:R_0603_1608Metric, F.Cu at (87.9, 124.9)
- added R15: 10k, Resistor_SMD:R_0603_1608Metric, F.Cu at (75.4, 124.9)
- added R16: 10k, Resistor_SMD:R_0603_1608Metric, B.Cu at (100.4, 124.9)
- added R16: 10k, Resistor_SMD:R_0603_1608Metric, B.Cu at (87.9, 124.9)
- added R16: 10k, Resistor_SMD:R_0603_1608Metric, B.Cu at (75.4, 124.9)
- added R17: 0, Resistor_SMD:R_0603_1608Metric, F.Cu at (103.0, 120.0)
- added R17: 0, Resistor_SMD:R_0603_1608Metric, F.Cu at (90.5, 120.0)
- added R17: 0, Resistor_SMD:R_0603_1608Metric, F.Cu at (78.0, 120.0)
- added R18: 0, Resistor_SMD:R_0603_1608Metric, B.Cu at (97.9, 120.0)
- added R18: 0, Resistor_SMD:R_0603_1608Metric, B.Cu at (85.4, 120.0)
- added R18: 0, Resistor_SMD:R_0603_1608Metric, B.Cu at (72.9, 120.0)
- added R19: 0, Resistor_SMD:R_0603_1608Metric, F.Cu at (97.9, 127.3)
- added R19: 0, Resistor_SMD:R_0603_1608Metric, F.Cu at (85.4, 127.3)
- added R19: 0, Resistor_SMD:R_0603_1608Metric, F.Cu at (72.9, 127.3)
- added R2: 2.2M, Resistor_SMD:R_0603_1608Metric, F.Cu at (103.0, 113.8)
- added R2: 2.2M, Resistor_SMD:R_0603_1608Metric, F.Cu at (90.5, 113.8)
- added R2: 2.2M, Resistor_SMD:R_0603_1608Metric, F.Cu at (78.0, 113.8)
- added R20: 0, Resistor_SMD:R_0603_1608Metric, B.Cu at (103.0, 127.2)
- added R20: 0, Resistor_SMD:R_0603_1608Metric, B.Cu at (90.5, 127.2)
- added R20: 0, Resistor_SMD:R_0603_1608Metric, B.Cu at (78.0, 127.2)
- added R21: 2.2M, Resistor_SMD:R_0603_1608Metric, F.Cu at (97.9, 120.0)
- added R21: 2.2M, Resistor_SMD:R_0603_1608Metric, F.Cu at (85.4, 120.0)
- added R21: 2.2M, Resistor_SMD:R_0603_1608Metric, F.Cu at (72.9, 120.0)
- added R22: 2.2M, Resistor_SMD:R_0603_1608Metric, B.Cu at (103.0, 120.0)
- added R22: 2.2M, Resistor_SMD:R_0603_1608Metric, B.Cu at (90.5, 120.0)
- added R22: 2.2M, Resistor_SMD:R_0603_1608Metric, B.Cu at (78.0, 120.0)
- added R23: 2.2M, Resistor_SMD:R_0603_1608Metric, F.Cu at (103.0, 127.2)
- added R23: 2.2M, Resistor_SMD:R_0603_1608Metric, F.Cu at (90.5, 127.2)
- added R23: 2.2M, Resistor_SMD:R_0603_1608Metric, F.Cu at (78.0, 127.2)
- added R24: 2.2M, Resistor_SMD:R_0603_1608Metric, B.Cu at (97.9, 127.2)
- added R24: 2.2M, Resistor_SMD:R_0603_1608Metric, B.Cu at (85.4, 127.2)
- added R24: 2.2M, Resistor_SMD:R_0603_1608Metric, B.Cu at (72.9, 127.2)
- added R3: 2.2M, Resistor_SMD:R_0603_1608Metric, F.Cu at (97.8, 106.5)
- added R3: 2.2M, Resistor_SMD:R_0603_1608Metric, F.Cu at (85.3, 106.5)
- added R3: 2.2M, Resistor_SMD:R_0603_1608Metric, F.Cu at (72.8, 106.5)
- added R4: 2.2M, Resistor_SMD:R_0603_1608Metric, B.Cu at (103.0, 106.5)
- added R4: 2.2M, Resistor_SMD:R_0603_1608Metric, B.Cu at (90.5, 106.5)
- added R4: 2.2M, Resistor_SMD:R_0603_1608Metric, B.Cu at (78.0, 106.5)
- added R5: 0, Resistor_SMD:R_0603_1608Metric, B.Cu at (103.0, 113.8)
- added R5: 0, Resistor_SMD:R_0603_1608Metric, B.Cu at (90.5, 113.8)
- added R5: 0, Resistor_SMD:R_0603_1608Metric, B.Cu at (78.0, 113.8)
- added R6: 0, Resistor_SMD:R_0603_1608Metric, F.Cu at (97.8, 113.8)
- added R6: 0, Resistor_SMD:R_0603_1608Metric, F.Cu at (85.3, 113.8)
- added R6: 0, Resistor_SMD:R_0603_1608Metric, F.Cu at (72.8, 113.8)
- added R7: 0, Resistor_SMD:R_0603_1608Metric, F.Cu at (103.0, 106.5)
- added R7: 0, Resistor_SMD:R_0603_1608Metric, F.Cu at (90.5, 106.5)
- added R7: 0, Resistor_SMD:R_0603_1608Metric, F.Cu at (78.0, 106.5)
- added R8: 0, Resistor_SMD:R_0603_1608Metric, B.Cu at (97.8, 106.5)
- added R8: 0, Resistor_SMD:R_0603_1608Metric, B.Cu at (85.3, 106.5)
- added R8: 0, Resistor_SMD:R_0603_1608Metric, B.Cu at (72.8, 106.5)
- added R9: 10k, Resistor_SMD:R_0603_1608Metric, B.Cu at (100.4, 111.4)
- added R9: 10k, Resistor_SMD:R_0603_1608Metric, B.Cu at (87.9, 111.4)
- added R9: 10k, Resistor_SMD:R_0603_1608Metric, B.Cu at (75.4, 111.4)
- added REF**: MountingHole_D1.524mm, Modules:MountingHole_D1.524mm, F.Cu at (105.4, 116.9)
- added REF**: MountingHole_2.29x3.81mm, Modules:MountingHole_2.29x3.81mm, F.Cu at (81.8, 89.4)
- added REF**: MountingHole_2.29x3.81mm, Modules:MountingHole_2.29x3.81mm, F.Cu at (74.3, 89.4)
- added REF**: MountingHole_D2.0mm, Modules:MountingHole_D2.0mm, F.Cu at (71.8, 91.8)
- added REF**: MountingHole_D2.0mm, Modules:MountingHole_D2.0mm, F.Cu at (71.8, 97.0)
- added REF**: MountingHole_D2.0mm, Modules:MountingHole_D2.0mm, F.Cu at (71.9, 102.2)
- added REF**: MountingHole_D1.524mm, Modules:MountingHole_D1.524mm, F.Cu at (67.9, 116.9)
- added REF**: MountingHole_D1.524mm, Modules:MountingHole_D1.524mm, F.Cu at (70.2, 116.9)
- added REF**: MountingHole_D1.524mm, Modules:MountingHole_D1.524mm, F.Cu at (92.9, 116.9)
- added REF**: MountingHole_D1.524mm, Modules:MountingHole_D1.524mm, F.Cu at (80.4, 116.9)
- added REF**: MountingHole_D1.524mm, Modules:MountingHole_D1.524mm, F.Cu at (107.7, 116.9)
- added REF**: MountingHole_D1.524mm, Modules:MountingHole_D1.524mm, F.Cu at (95.2, 116.9)
- added REF**: MountingHole_D1.524mm, Modules:MountingHole_D1.524mm, F.Cu at (82.7, 116.9)
- added REF**: MountingHole_2.29x5.46mm, Modules:MountingHole_2.29x5.46mm, F.Cu at (105.2, 83.3)
- added REF**: MountingHole_2.29x3.81mm, Modules:MountingHole_2.29x3.81mm, F.Cu at (102.4, 89.4)
- added REF**: MountingHole_2.29x3.81mm, Modules:MountingHole_2.29x3.81mm, F.Cu at (94.8, 89.4)
- added U1: ADuM1251ARZ, Package_SO:SOIC-8_3.9x4.9mm_P1.27mm, B.Cu at (106.6, 116.9)
- added U1: ADuM1251ARZ, Package_SO:SOIC-8_3.9x4.9mm_P1.27mm, B.Cu at (94.1, 116.9)
- added U1: ADuM1251ARZ, Package_SO:SOIC-8_3.9x4.9mm_P1.27mm, B.Cu at (81.6, 116.9)
- added U2: ADuM1201AR, Package_SO:SOIC-8_3.9x4.9mm_P1.27mm, F.Cu at (106.6, 116.9)
- added U2: ADuM1201AR, Package_SO:SOIC-8_3.9x4.9mm_P1.27mm, F.Cu at (94.1, 116.9)
- added U2: ADuM1201AR, Package_SO:SOIC-8_3.9x4.9mm_P1.27mm, F.Cu at (81.6, 116.9)
- moved C1 11.4 mm to (93.0, 57.6)
- moved C1 11.4 mm to (69.1, 110.2)
- moved C10 11.4 mm to (92.3, 68.1)
- moved C12 11.4 mm to (102.2, 68.1)
- moved C13 11.4 mm to (84.6, 72.9)
- moved C13 11.4 mm to (89.7, 83.2)
- moved C14 11.4 mm to (80.8, 72.2)
- moved C16 11.4 mm to (86.8, 65.5)
- moved C17 11.4 mm to (76.0, 62.5)
- moved C19 11.4 mm to (82.2, 55.3)
- moved C2 11.4 mm to (69.1, 111.7)
- moved C3 11.4 mm to (76.0, 81.1)
- moved C3 11.4 mm to (69.1, 111.7)
- moved C4 11.4 mm to (69.1, 122.1)
- moved C5 11.4 mm to (78.7, 55.3)
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Routing:
- net Net-(Q4-Pad2): track 81.3 -> 36.9 mm
- net /SDA: track 60.4 -> 33.1 mm
- net /SCL: track 68.0 -> 45.0 mm
- net VCCQ: track 157.9 -> 175.8 mm
- net /SCLq: track 86.2 -> 70.1 mm
- net Net-(Q2-Pad2): track 54.9 -> 39.7 mm
- net Net-(Q3-Pad2): track 62.0 -> 49.1 mm
- net /outa: track 33.2 -> 44.3 mm
- net Net-(Q7-Pad2): track 62.8 -> 53.1 mm
- net /inb: track 41.1 -> 50.2 mm
- net Net-(Q5-Pad2): track 40.9 -> 46.7 mm
- net Net-(Q8-Pad2): track 56.0 -> 59.5 mm
- net Net-(Q1-Pad2): track 36.4 -> 33.8 mm
- net Net-(Q6-Pad2): track 60.2 -> 62.1 mm
- net /SDAq: track 63.9 -> 64.9 mm
Other:
- board text removed: "JLCJLCJLCJLC"
